File: hardware/Diag6502rp/_autosave-Diag6502rp.kicad_pcb (KiCad board)
At the start: 4 copper layers, 59.5 x 54.3 mm, 83 parts, among them J1 Conn_01x20_PinHeader, J10 Conn_01x20_PinHeader, J11 Conn_01x20_PinHeader, J2 Conn_01x20_PinSocket, J3 Conn_01x20_PinHeader, J4 Conn_01x20_PinSocket, J5 GT-USB-7010AN, J6 Conn_02x20_Counter_Clockwise, J7 Conn_ARM_SWD_TagConnect_TC2030, J8 Conn_01x02_PinSocket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

Commit message: Added transfer and stitching vias.
Parts:
- moved SW1 1.00 mm to (131.3, 39.6)
- moved D2 0.07 mm to (147.2, 50.9)
Routing:
- net Net-(R7-Pad1): track 8.32 -> 10.2 mm
- net /Processor/PHI2: track 26.1 -> 27.5 mm
- net /Processor/QSPI_SS: track 20.7 -> 20.2 mm
- net +3V3: track 50.1 -> 49.6 mm, vias 24 -> 25
- net GND: track 47.6 -> 47.3 mm, vias 88 -> 101
Other:
- board text added: "Diag6502 Logic-Board"
